Commit message: Signed-off-by: Andrea Patrizi <andreapatrizi1b6e6@gmail.com>

File: robots/aliengo_description/aliengo_srdf/srdf/aliengo.srdf.xacro (robot description, xacro)
@@ -6,6 +6,4 @@
 <robot xmlns:xacro="http://ros.org/wiki/xacro" name="kyon">
     <!-- ************ MODEL CONFIGURATION ************ -->
-    <xacro:arg name="config" default="$(find kyon_urdf)/urdf/config/kyon.urdf.xacro"/>
-    <xacro:include filename="$(arg config)"/>
     <group name="base">
         <link name="pelvis"/>

File: robots/aliengo_description/aliengo_urdf/urdf/aliengo.urdf.xacro (robot description, xacro)
@@ -1,7 +1,11 @@
 <?xml version="1.0"?>
 <robot name="aliengo" xmlns:xacro="http://www.ros.org/wiki/xacro">
-    <xacro:include filename="$(find aliengo_urdf)/urdf/const.xacro"/>
-    <xacro:include filename="$(find aliengo_urdf)/urdf/materials.xacro"/>
-    <xacro:include filename="$(find aliengo_urdf)/urdf/leg.xacro"/>
+    <!-- This argument and property should be in the top level xacro and
+    will be propagated to all its downstream childs -->
+    <xacro:arg name="aliengo_root" default="$(find aliengo_urdf)" />
+    <xacro:property name="ALIENGO_ROOT" value="$(arg aliengo_root)" />
+    <xacro:include filename="${ALIENGO_ROOT}/urdf/const.xacro"/>
+    <xacro:include filename="${ALIENGO_ROOT}/urdf/materials.xacro"/>
+    <xacro:include filename="${ALIENGO_ROOT}/urdf/leg.xacro"/>
     <!-- <xacro:include filename="$(find aliengo_urdf)/urdf/gazebo.xacro"/> -->
     <!-- Rotor related joint and link is only for demonstrate location. -->
@@ -18,5 +22,5 @@
             <origin rpy="0 0 0" xyz="0 0 0"/>
             <geometry>
-                <mesh filename="package://aliengo_urdf/meshes/trunk.dae" scale="1 1 1"/>
+                <mesh filename="${ALIENGO_ROOT}/meshes/trunk.dae" scale="1 1 1"/>
             </geometry>
             <material name="orange"/>
@@ -31,5 +35,5 @@
             <origin rpy="0 0 0" xyz="0 0 0"/>
             <geometry>
-                <mesh filename="package://aliengo_urdf/meshes/trunk.dae" scale="1 1 1"/>
+                <mesh filename="${ALIENGO_ROOT}/meshes/trunk.dae" scale="1 1 1"/>
             </geometry>
         </collision> -->

File: robots/aliengo_description/aliengo_urdf/urdf/leg.xacro (robot description, xacro)
@@ -1,5 +1,5 @@
 <?xml version="1.0"?>
 <robot xmlns:xacro="http://www.ros.org/wiki/xacro">
-    <xacro:include filename="$(find aliengo_urdf)/urdf/transmission.xacro"/>
+    <xacro:include filename="${ALIENGO_ROOT}/urdf/transmission.xacro"/>
     <xacro:macro name="leg" params="name mirror mirror_dae front_hind front_hind_dae">
         <joint name="${name}_hip_joint" type="revolute">
@@ -58,5 +58,5 @@
                 </xacro:if>
                 <geometry>
-                    <mesh filename="package://aliengo_urdf/meshes/hip.dae" scale="1 1 1"/>
+                    <mesh filename="${ALIENGO_ROOT}/meshes/hip.dae" scale="1 1 1"/>
                 </geometry>
                 <material name="orange"/>
@@ -118,8 +118,8 @@
                 <geometry>
                     <xacro:if value="${mirror_dae == True}">
-                        <mesh filename="package://aliengo_urdf/meshes/thigh.dae" scale="1 1 1"/>
+                        <mesh filename="${ALIENGO_ROOT}/meshes/thigh.dae" scale="1 1 1"/>
                     </xacro:if>
                     <xacro:if value="${mirror_dae == False}">
-                        <mesh filename="package://aliengo_urdf/meshes/thigh_mirror.dae" scale="1 1 1"/>
+                        <mesh filename="${ALIENGO_ROOT}/meshes/thigh_mirror.dae" scale="1 1 1"/>
                     </xacro:if>
                 </geometry>
