Commit message: Signed-off-by: Andrea Patrizi <andreapatrizi1b6e6@gmail.com>

File: robots/aliengo_description/aliengo_urdf/urdf/leg.xacro (robot description, xacro)
@@ -181,5 +181,5 @@
                 <origin rpy="0 0 0" xyz="0 0 0"/>
                 <geometry>
-                    <mesh filename="package://aliengo_urdf/meshes/calf.dae" scale="1 1 1"/>
+                    <mesh filename="${MESH_PATH}/calf.dae" scale="1 1 1"/>
                 </geometry>
                 <material name="orange"/>
