Commit message: modified aliengo_description layout

File: robots/aliengo_description/aliengo_urdf/urdf/aliengo.urdf.xacro (robot description, xacro)
@@ -1,31 +1,16 @@
 <?xml version="1.0"?>
 <robot name="aliengo" xmlns:xacro="http://www.ros.org/wiki/xacro">
-    <xacro:include filename="$(find aliengo_description)/xacro/const.xacro"/>
-    <xacro:include filename="$(find aliengo_description)/xacro/materials.xacro"/>
-    <xacro:include filename="$(find aliengo_description)/xacro/leg.xacro"/>
-    <xacro:include filename="$(find aliengo_description)/xacro/gazebo.xacro"/>
+    <xacro:include filename="$(find aliengo_urdf)/urdf/const.xacro"/>
+    <xacro:include filename="$(find aliengo_urdf)/urdf/materials.xacro"/>
+    <xacro:include filename="$(find aliengo_urdf)/urdf/leg.xacro"/>
+    <!-- <xacro:include filename="$(find aliengo_urdf)/urdf/gazebo.xacro"/> -->
     <!-- Rotor related joint and link is only for demonstrate location. -->
     <!-- Actually, the rotor will rotate and the joint is not fixed. Reduction ratio should be considered. -->
     <!-- Debug mode will hung up the robot, use "true" or "false" to switch it. -->
-    <xacro:if value="$(arg DEBUG)">
-        <link name="world"/>
-        <joint name="base_static_joint" type="fixed">
-            <origin rpy="0 0 0" xyz="0 0 0"/>
-            <parent link="world"/>
-            <child link="base"/>
-        </joint>
-    </xacro:if>
-    <link name="base">
-        <visual>
-            <origin rpy="0 0 0" xyz="0 0 0"/>
-            <geometry>
-                <box size="0.001 0.001 0.001"/>
-            </geometry>
-        </visual>
-    </link>
-    <joint name="floating_base" type="fixed">
-        <origin rpy="0 0 0" xyz="0 0 0"/>
-        <parent link="base"/>
+    <link name="base_link"/>
+    <joint name="base_joint" type="fixed">
+        <parent link="base_link"/>
         <child link="trunk"/>
+        <origin xyz="0 0 0" rpy="0 0 0" />
     </joint>
     <link name="trunk">
@@ -33,5 +18,5 @@
             <origin rpy="0 0 0" xyz="0 0 0"/>
             <geometry>
-                <mesh filename="package://aliengo_description/meshes/trunk.dae" scale="1 1 1"/>
+                <mesh filename="package://aliengo_urdf/meshes/trunk.dae" scale="1 1 1"/>
             </geometry>
             <material name="orange"/>
@@ -46,5 +31,5 @@
             <origin rpy="0 0 0" xyz="0 0 0"/>
             <geometry>
-                <mesh filename="package://aliengo_description/meshes/trunk.dae" scale="1 1 1"/>
+                <mesh filename="package://aliengo_urdf/meshes/trunk.dae" scale="1 1 1"/>
             </geometry>
         </collision> -->

File: robots/aliengo_description/aliengo_urdf/urdf/leg.xacro (robot description, xacro)
@@ -1,5 +1,5 @@
 <?xml version="1.0"?>
 <robot xmlns:xacro="http://www.ros.org/wiki/xacro">
-    <xacro:include filename="$(find aliengo_description)/xacro/transmission.xacro"/>
+    <xacro:include filename="$(find aliengo_urdf)/urdf/transmission.xacro"/>
     <xacro:macro name="leg" params="name mirror mirror_dae front_hind front_hind_dae">
         <joint name="${name}_hip_joint" type="revolute">
@@ -58,5 +58,5 @@
                 </xacro:if>
                 <geometry>
-                    <mesh filename="package://aliengo_description/meshes/hip.dae" scale="1 1 1"/>
+                    <mesh filename="package://aliengo_urdf/meshes/hip.dae" scale="1 1 1"/>
                 </geometry>
                 <material name="orange"/>
@@ -100,5 +100,5 @@
             </inertial>
         </link>
-        <joint name="${name}_thigh_joint" type="continuous">
+        <joint name="${name}_thigh_joint" type="revolute">
             <origin rpy="0 0 0" xyz="0 ${thigh_offset*mirror} 0"/>
             <parent link="${name}_hip"/>
@@ -118,8 +118,8 @@
                 <geometry>
                     <xacro:if value="${mirror_dae == True}">
-                        <mesh filename="package://aliengo_description/meshes/thigh.dae" scale="1 1 1"/>
+                        <mesh filename="package://aliengo_urdf/meshes/thigh.dae" scale="1 1 1"/>
                     </xacro:if>
                     <xacro:if value="${mirror_dae == False}">
-                        <mesh filename="package://aliengo_description/meshes/thigh_mirror.dae" scale="1 1 1"/>
+                        <mesh filename="package://aliengo_urdf/meshes/thigh_mirror.dae" scale="1 1 1"/>
                     </xacro:if>
                 </geometry>
@@ -181,5 +181,5 @@
                 <origin rpy="0 0 0" xyz="0 0 0"/>
                 <geometry>
-                    <mesh filename="package://aliengo_description/meshes/calf.dae" scale="1 1 1"/>
+                    <mesh filename="package://aliengo_urdf/meshes/calf.dae" scale="1 1 1"/>
                 </geometry>
                 <material name="orange"/>

File: robots/aliengo_description/aliengo_urdf/urdf/prova.urdf (robot description, URDF)
Before this commit: robot aliengo, 31 links, 30 joints
Links:
- removed link base
- removed link trunk
- added link pelvis, mass 11.644; collision box size=0.647 0.15 0.112; visual mesh filename=package://aliengo_urdf/meshes/trunk.dae scale=1 1 1
- link FL_calf: geometry collision box size=0.25 0.0208 0.016; visual mesh filename=package://aliengo_urdf/meshes/calf.dae scale=1 1 1
- link FL_calf_rotor: geometry visual cylinder length=0.02 radius=0.035
- link FL_hip: geometry collision cylinder length=0.0418 radius=0.046; visual mesh filename=package://aliengo_urdf/meshes/hip.dae scale=1 1 1
- link FL_hip_rotor: geometry visual cylinder length=0.02 radius=0.035
- link FL_thigh: geometry collision box size=0.25 0.0374 0.043; visual mesh filename=package://aliengo_urdf/meshes/thigh.dae scale=1 1 1
- link FL_thigh_rotor: geometry visual cylinder length=0.02 radius=0.035
- link FR_calf: geometry collision box size=0.25 0.0208 0.016; visual mesh filename=package://aliengo_urdf/meshes/calf.dae scale=1 1 1
- link FR_calf_rotor: geometry visual cylinder length=0.02 radius=0.035
- link FR_hip: geometry collision cylinder length=0.0418 radius=0.046; visual mesh filename=package://aliengo_urdf/meshes/hip.dae scale=1 1 1
- link FR_hip_rotor: geometry visual cylinder length=0.02 radius=0.035
- link FR_thigh: geometry collision box size=0.25 0.0374 0.043; visual mesh filename=package://aliengo_urdf/meshes/thigh_mirror.dae scale=1 1 1
- link FR_thigh_rotor: geometry visual cylinder length=0.02 radius=0.035
- link RL_calf: geometry collision box size=0.25 0.0208 0.016; visual mesh filename=package://aliengo_urdf/meshes/calf.dae scale=1 1 1
- link RL_calf_rotor: geometry visual cylinder length=0.02 radius=0.035
- link RL_hip: geometry collision cylinder length=0.0418 radius=0.046; visual mesh filename=package://aliengo_urdf/meshes/hip.dae scale=1 1 1
- link RL_hip_rotor: geometry visual cylinder length=0.02 radius=0.035
- link RL_thigh: geometry collision box size=0.25 0.0374 0.043; visual mesh filename=package://aliengo_urdf/meshes/thigh.dae scale=1 1 1
- link RL_thigh_rotor: geometry visual cylinder length=0.02 radius=0.035
- link RR_calf: geometry collision box size=0.25 0.0208 0.016; visual mesh filename=package://aliengo_urdf/meshes/calf.dae scale=1 1 1
- link RR_calf_rotor: geometry visual cylinder length=0.02 radius=0.035
- link RR_hip: geometry collision cylinder length=0.0418 radius=0.046; visual mesh filename=package://aliengo_urdf/meshes/hip.dae scale=1 1 1
- link RR_hip_rotor: geometry visual cylinder length=0.02 radius=0.035
- link RR_thigh: geometry collision box size=0.25 0.0374 0.043; visual mesh filename=package://aliengo_urdf/meshes/thigh_mirror.dae scale=1 1 1
- link RR_thigh_rotor: geometry visual cylinder length=0.02 radius=0.035
Joints:
- removed joint floating_base
- joint FL_thigh_joint: type continuous -> revolute
- joint FR_thigh_joint: type continuous -> revolute
- joint RL_thigh_joint: type continuous -> revolute
- joint RR_thigh_joint: type continuous -> revolute

Commit message: Signed-off-by: Andrea Patrizi <andreapatrizi1b6e6@gmail.com>

File: robots/aliengo_description/aliengo_urdf/urdf/aliengo.urdf.xacro (robot description, xacro)
@@ -5,4 +5,15 @@
     <xacro:arg name="aliengo_root" default="$(find aliengo_urdf)" />
     <xacro:property name="ALIENGO_ROOT" value="$(arg aliengo_root)" />
+    <!-- setting use_abs_mesh_paths should be kept to false
+    for use with tools like RViz, which does not accept plain
+    abolute paths for mesh paths-->
+    <xacro:arg name="use_abs_mesh_paths" default="false" />
+    <xacro:property name="USE_ABS_MESH_PATHS" value="$(arg use_abs_mesh_paths)" />
+    <xacro:if value="${USE_ABS_MESH_PATHS}">
+    <xacro:property name="MESH_PATH" value="${ALIENGO_ROOT}/meshes" />
+    </xacro:if>
+    <xacro:unless value="${USE_ABS_MESH_PATHS}">
+    <xacro:property name="MESH_PATH" value="package://aliengo_urdf/meshes" />
+    </xacro:unless>
     <xacro:include filename="${ALIENGO_ROOT}/urdf/const.xacro"/>
     <xacro:include filename="${ALIENGO_ROOT}/urdf/materials.xacro"/>
@@ -22,5 +33,5 @@
             <origin rpy="0 0 0" xyz="0 0 0"/>
             <geometry>
-                <mesh filename="${ALIENGO_ROOT}/meshes/trunk.dae" scale="1 1 1"/>
+                <mesh filename="${MESH_PATH}/trunk.dae" scale="1 1 1"/>
             </geometry>
             <material name="orange"/>
@@ -35,5 +46,5 @@
             <origin rpy="0 0 0" xyz="0 0 0"/>
             <geometry>
-                <mesh filename="${ALIENGO_ROOT}/meshes/trunk.dae" scale="1 1 1"/>
+                <mesh filename="${MESH_PATH}/trunk.dae" scale="1 1 1"/>
             </geometry>
         </collision> -->

File: robots/aliengo_description/aliengo_urdf/urdf/leg.xacro (robot description, xacro)
@@ -58,5 +58,5 @@
                 </xacro:if>
                 <geometry>
-                    <mesh filename="${ALIENGO_ROOT}/meshes/hip.dae" scale="1 1 1"/>
+                    <mesh filename="${MESH_PATH}/hip.dae" scale="1 1 1"/>
                 </geometry>
                 <material name="orange"/>
@@ -118,8 +118,8 @@
                 <geometry>
                     <xacro:if value="${mirror_dae == True}">
-                        <mesh filename="${ALIENGO_ROOT}/meshes/thigh.dae" scale="1 1 1"/>
+                        <mesh filename="${MESH_PATH}/thigh.dae" scale="1 1 1"/>
                     </xacro:if>
                     <xacro:if value="${mirror_dae == False}">
-                        <mesh filename="${ALIENGO_ROOT}/meshes/thigh_mirror.dae" scale="1 1 1"/>
+                        <mesh filename="${MESH_PATH}/thigh_mirror.dae" scale="1 1 1"/>
                     </xacro:if>
                 </geometry>

Commit message: added flag to allow use with abs paths and rviz

File: robots/aliengo_description/aliengo_urdf/urdf/aliengo.urdf.xacro (robot description, xacro)
@@ -9,8 +9,15 @@
     abolute paths for mesh paths-->
     <xacro:arg name="use_abs_mesh_paths" default="false" />
+    <xacro:arg name="use_local_filesys_for_meshes" default="false" />
     <xacro:property name="USE_ABS_MESH_PATHS" value="$(arg use_abs_mesh_paths)" />
+    <xacro:property name="USE_LOCAL_FILESYS_FOR_MESHES" value="$(arg use_local_filesys_for_meshes)" />
     <xacro:if value="${USE_ABS_MESH_PATHS}">
-    <xacro:property name="MESH_PATH" value="${ALIENGO_ROOT}/meshes" />
-    </xacro:if>
+        <xacro:if value="${USE_LOCAL_FILESYS_FOR_MESHES}">
+        <xacro:property name="MESH_PATH" value="file://${ALIENGO_ROOT}/meshes" />
+        </xacro:if>
+        <xacro:unless value="${USE_ABS_MESH_PATHS}">
+        <xacro:property name="MESH_PATH" value="${ALIENGO_ROOT}/meshes" />
+        </xacro:unless>
+        </xacro:if>
     <xacro:unless value="${USE_ABS_MESH_PATHS}">
     <xacro:property name="MESH_PATH" value="package://aliengo_urdf/meshes" />
