Commit message: added srdf + complied with IBRIDO descr specs

File: robots/b2w_description/urdf/b2w_description.urdf (robot description, URDF)
Before this commit: robot b2w_description, 26 links, 25 joints
Links:
- link FL_calf: geometry collision mesh filename=${MESH_PATH}/FL_calf.dae; visual mesh filename=${MESH_PATH}/FL_calf.dae
- link FL_foot: geometry collision mesh filename=${MESH_PATH}/FL_foot.dae; visual mesh filename=${MESH_PATH}/FL_foot.dae
- link FL_hip: geometry collision cylinder length=0.05 radius=0.07; visual mesh filename=${MESH_PATH}/FL_hip.dae
- link FL_thigh: geometry collision box size=0.32 0.0445 0.054; visual mesh filename=${MESH_PATH}/FL_thigh.dae
- link FR_calf: geometry collision mesh filename=${MESH_PATH}/FR_calf.dae; visual mesh filename=${MESH_PATH}/FR_calf.dae
- link FR_foot: geometry collision mesh filename=${MESH_PATH}/FR_foot.dae; visual mesh filename=${MESH_PATH}/FR_foot.dae
- link FR_hip: geometry collision cylinder length=0.05 radius=0.07; visual mesh filename=${MESH_PATH}/FR_hip.dae
- link FR_thigh: geometry collision box size=0.25 0.028 0.04; visual mesh filename=${MESH_PATH}/FR_thigh.dae
- link RL_calf: geometry collision mesh filename=${MESH_PATH}/RL_calf.dae; visual mesh filename=${MESH_PATH}/RL_calf.dae
- link RL_foot: geometry collision mesh filename=${MESH_PATH}/RL_foot.dae; visual mesh filename=${MESH_PATH}/RL_foot.dae
- link RL_hip: geometry collision cylinder length=0.05 radius=0.07; visual mesh filename=${MESH_PATH}/RL_hip.dae
- link RL_thigh: geometry collision box size=0.25 0.028 0.04; visual mesh filename=${MESH_PATH}/RL_thigh.dae
- link RR_calf: geometry collision mesh filename=${MESH_PATH}/RR_calf.dae; visual mesh filename=${MESH_PATH}/RR_calf.dae
- link RR_foot: geometry collision mesh filename=${MESH_PATH}/RR_foot.dae; visual mesh filename=${MESH_PATH}/RR_foot.dae
- link RR_hip: geometry collision cylinder length=0.05 radius=0.07; visual mesh filename=${MESH_PATH}/RR_hip.dae
- link RR_thigh: geometry collision box size=0.25 0.028 0.04; visual mesh filename=${MESH_PATH}/RR_thigh.dae
- link base_link: geometry collision box size=0.5 0.28 0.15; visual mesh filename=${MESH_PATH}/base_link.dae

File: robots/b2w_description/xacro/leg.xacro (robot description, xacro)
@@ -1,5 +1,5 @@
 <?xml version="1.0"?>
 <robot xmlns:xacro="http://www.ros.org/wiki/xacro">
-    <xacro:include filename="$(find b2w_description)/xacro/transmission.xacro"/>
+    <xacro:include filename="${ROOT}/xacro/transmission.xacro"/>
     <xacro:macro name="leg" params="name mirror mirror_dae front_hind front_hind_dae">
         <joint name="${name}_hip_joint" type="revolute">
@@ -58,5 +58,5 @@
                 </xacro:if>
                 <geometry>
-                    <mesh filename="package://b2w_description/meshes/hip.dae" scale="1 1 1"/>
+                    <mesh filename="${MESH_PATH}/hip.dae" scale="1 1 1"/>
                 </geometry>
                 <material name="orange"/>
@@ -112,8 +112,8 @@
                 <geometry>
                     <xacro:if value="${mirror_dae == True}">
-                        <mesh filename="package://b2w_description/meshes/thigh.dae" scale="1 1 1"/>
+                        <mesh filename="${MESH_PATH}/thigh.dae" scale="1 1 1"/>
                     </xacro:if>
                     <xacro:if value="${mirror_dae == False}">
-                        <mesh filename="package://b2w_description/meshes/thigh_mirror.dae" scale="1 1 1"/>
+                        <mesh filename="${MESH_PATH}/thigh_mirror.dae" scale="1 1 1"/>
                     </xacro:if>
                 </geometry>
@@ -170,8 +170,8 @@
                 <geometry>
                     <xacro:if value="${mirror_dae == True}">
-                        <mesh filename="package://b2w_description/meshes/thigh.dae" scale="1 1 1"/>
+                        <mesh filename="${MESH_PATH}/thigh.dae" scale="1 1 1"/>
                     </xacro:if>
                     <xacro:if value="${mirror_dae == False}">
-                        <mesh filename="package://b2w_description/meshes/thigh_mirror.dae" scale="1 1 1"/>
+                        <mesh filename="${MESH_PATH}/thigh_mirror.dae" scale="1 1 1"/>
                     </xacro:if>
                 </geometry>
@@ -182,8 +182,8 @@
                 <geometry>
                     <xacro:if value="${mirror_dae == True}">
-                        <mesh filename="package://b2w_description/meshes/calf.dae" scale="1 1 1"/>
+                        <mesh filename="${MESH_PATH}/calf.dae" scale="1 1 1"/>
                     </xacro:if>
                     <xacro:if value="${mirror_dae == False}">
-                        <mesh filename="package://b2w_description/meshes/calf_mirror.dae" scale="1 1 1"/>
+                        <mesh filename="${MESH_PATH}/calf_mirror.dae" scale="1 1 1"/>
                     </xacro:if>
                 </geometry>

File: robots/b2w_description/xacro/robot.urdf.xacro (robot description, xacro)
@@ -1,12 +1,31 @@
 <?xml version="1.0"?>
-<robot name="b2w_description" xmlns:xacro="http://www.ros.org/wiki/xacro">
-    <xacro:include filename="$(find b2w_description)/xacro/const.xacro"/>
-    <xacro:include filename="$(find b2w_description)/xacro/materials.xacro"/>
-    <xacro:include filename="$(find b2w_description)/xacro/leg.xacro"/>
-    <xacro:include filename="$(find b2w_description)/xacro/gazebo.xacro"/>
+<robot name="unitree_b2w" xmlns:xacro="http://www.ros.org/wiki/xacro">
+    <xacro:arg name="debug" default="false" />
+    <xacro:property name="DEBUG" value="$(arg debug)" />
+    <xacro:arg name="root" default="${ROOT}" />
+    <xacro:arg name="use_abs_mesh_paths" default="false" />
+    <xacro:arg name="use_local_filesys_for_meshes" default="false" />
+    <xacro:property name="ROOT" value="$(arg root)" />
+    <xacro:property name="USE_ABS_MESH_PATHS" value="$(arg use_abs_mesh_paths)" />
+    <xacro:property name="USE_LOCAL_FILESYS_FOR_MESHES" value="$(arg use_local_filesys_for_meshes)" />
+    <xacro:if value="${USE_ABS_MESH_PATHS}">
+        <xacro:if value="${USE_LOCAL_FILESYS_FOR_MESHES}">
+        <xacro:property name="MESH_PATH" value="file://${ROOT}/meshes" />
+        </xacro:if>
+        <xacro:unless value="${USE_LOCAL_FILESYS_FOR_MESHES}">
+        <xacro:property name="MESH_PATH" value="${ROOT}/meshes" />
+        </xacro:unless>
+    </xacro:if>
+    <xacro:unless value="${USE_ABS_MESH_PATHS}">
+        <xacro:property name="MESH_PATH" value="package://b2w_description/meshes" />
+    </xacro:unless>
+    <xacro:include filename="${ROOT}/xacro/const.xacro"/>
+    <xacro:include filename="${ROOT}/xacro/materials.xacro"/>
+    <xacro:include filename="${ROOT}/xacro/leg.xacro"/>
+    <xacro:include filename="${ROOT}/xacro/gazebo.xacro"/>
     <!-- Rotor related joint and link is only for demonstrate location. -->
     <!-- Actually, the rotor will rotate and the joint is not fixed. Reduction ratio should be considered. -->
     <!-- Debug mode will hung up the robot, use "true" or "false" to switch it. -->
-    <xacro:if value="$(arg DEBUG)">
+    <xacro:if value="${DEBUG}">
         <link name="world"/>
         <joint name="base_static_joint" type="fixed">
@@ -33,5 +52,5 @@
             <origin rpy="0 0 0" xyz="0 0 0"/>
             <geometry>
-                <mesh filename="package://b2w_description/meshes/trunk.dae" scale="1 1 1"/>
+                <mesh filename="${MESH_PATH}/trunk.dae" scale="1 1 1"/>
             </geometry>
             <!-- <material name="orange"/> -->
