Commit message: Signed-off-by: Andrea Patrizi <andreapatrizi1b6e6@gmail.com>

File: robots/b2w_description/xacro/robot.srdf.xacro (robot description, xacro)
@@ -9,5 +9,5 @@
     <xacro:property name="ROOT" value="$(arg root)" />
     <group name="base">
-        <link name="base"/>base_link
+        <link name="base"/>
     </group>
     <group name="imu_sensors">
@@ -25,4 +25,10 @@
     <group name="rear_left_leg">
         <chain base="base" tip_link="RL_foot" />
+    </group>
+    <group name="chains">
+        <group name="front_left_leg"/>
+        <group name="front_right_leg"/>
+        <group name="rear_right_leg"/>
+        <group name="rear_left_leg"/>
     </group>
     <!-- Homing posture -->
