Commit message: Signed-off-by: Andrea Patrizi <andreapatrizi1b6e6@gmail.com>

File: robots/b2w_description/xacro/robot.urdf.xacro (robot description, xacro)
@@ -148,5 +148,5 @@
         <inertial>
             <origin rpy="0 0 0" xyz="0 0 0"/>
-            <mass value="6.55E-08" />
+            <mass value="1.0E-03" />
             <inertia
                 ixx="1e-3"
