Commit message: fixed missing wheels in xacro

File: robots/b2w_description/xacro/leg.xacro (robot description, xacro)
@@ -240,26 +240,57 @@
             </inertial>
         </link>
-        <joint name="${name}_foot_fixed" type="fixed">
-            <origin rpy="1.57 0 0" xyz="0 0 ${-(calf_length)}"/>
-            <parent link="${name}_calf"/>
-            <child link="${name}_foot"/>
-        </joint>
-        <link name="${name}_foot">
-            <collision>
-            <origin
-                xyz="0 0 0"
-                rpy="0 0 0" />
-            <geometry>
-                <sphere radius="0.032" />
-            </geometry>
-            </collision>
-            <inertial>
-                <mass value="${foot_mass}"/>
-                <inertia
-                    ixx="${(2*foot_mass)/5.0*(foot_radius*foot_radius)}" ixy="0.0" ixz="0.0"
-                    iyy="${(2*foot_mass)/5.0*(foot_radius*foot_radius)}" iyz="0.0"
-                    izz="${(2*foot_mass)/5.0*(foot_radius*foot_radius)}"/>
-            </inertial>
-        </link>
+        <xacro:if value="${ADD_WHEELS}">
+            <joint name="${name}_foot_joint" type="continuous">
+                <origin xyz="0 -0.001 -0.35" rpy="0 0 0" />
+                <parent link="${name}_calf" />
+                <child link="${name}_foot" />
+                <axis xyz="0 1 0" />
+                <limit effort="20" velocity="50" />
+            </joint>
+            <link name="${name}_foot">
+                <inertial>
+                    <origin xyz="-0.000991 -0.051053 -0.00113" rpy="0 0 0" />
+                    <mass value="1.083" />
+                    <inertia ixx="0.004121" ixy="-6E-06" ixz="-4.8E-05" iyy="0.007776" iyz="-7E-06" izz="0.004108" />
+                </inertial>
+                <visual>
+                    <origin xyz="0 0 0" rpy="0 0 0" />
+                    <geometry>
+                        <mesh filename="${MESH_PATH}/${name}_foot.dae" />
+                    </geometry>
+                    <material name="">
+                        <color rgba="1 1 1 1" />
+                    </material>
+                </visual>
+                <collision>
+                    <origin xyz="0 0 0" rpy="0 0 0" />
+                    <geometry>
+                        <mesh filename="${MESH_PATH}/${name}_foot.dae" />
+                    </geometry>
+                </collision>
+            </link>
+        </xacro:if>
+        <xacro:unless value="${ADD_WHEELS}">
+            <joint name="${name}_foot_fixed" type="fixed">
+                <origin rpy="1.57 0 0" xyz="0 0 ${-(calf_length)}"/>
+                <parent link="${name}_calf"/>
+                <child link="${name}_foot"/>
+            </joint>
+            <link name="${name}_foot">
+                <collision>
+                    <origin xyz="0 0 0" rpy="0 0 0" />
+                    <geometry>
+                        <sphere radius="0.032" />
+                    </geometry>
+                </collision>
+                <inertial>
+                    <mass value="${foot_mass}"/>
+                    <inertia
+                        ixx="${(2*foot_mass)/5.0*(foot_radius*foot_radius)}" ixy="0.0" ixz="0.0"
+                        iyy="${(2*foot_mass)/5.0*(foot_radius*foot_radius)}" iyz="0.0"
+                        izz="${(2*foot_mass)/5.0*(foot_radius*foot_radius)}"/>
+                </inertial>
+            </link>
+        </xacro:unless>
         <xacro:leg_transmission name="${name}"/>
     </xacro:macro>

File: robots/b2w_description/xacro/robot.urdf.xacro (robot description, xacro)
@@ -3,8 +3,12 @@
     <xacro:arg name="debug" default="false" />
     <xacro:property name="DEBUG" value="$(arg debug)" />
+    <xacro:arg name="floating_joint" default="false"/>
+    <xacro:arg name="wheels" default="true"/>
     <xacro:arg name="root" default="${ROOT}" />
     <xacro:arg name="use_abs_mesh_paths" default="false" />
     <xacro:arg name="use_local_filesys_for_meshes" default="false" />
     <xacro:property name="ROOT" value="$(arg root)" />
+    <xacro:property name="ADD_FLOATING_BASE" value="$(arg floating_joint)" />
+    <xacro:property name="ADD_WHEELS" value="$(arg wheels)" />
     <xacro:property name="USE_ABS_MESH_PATHS" value="$(arg use_abs_mesh_paths)" />
     <xacro:property name="USE_LOCAL_FILESYS_FOR_MESHES" value="$(arg use_local_filesys_for_meshes)" />
@@ -35,4 +39,14 @@
         </joint>
     </xacro:if>
+    <xacro:unless value="${DEBUG}">
+        <!-- add floating joint only if not DEBUG -->
+        <xacro:if value="${ADD_FLOATING_BASE}">
+            <link name="world"/>
+            <joint name="reference" type="floating">
+                <parent link="world"/>
+                <child link="base"/>
+            </joint>
+        </xacro:if>
+    </xacro:unless>
     <link name="base">
         <visual>
@@ -43,5 +57,5 @@
         </visual>
     </link>
-    <joint name="floating_base" type="fixed">
+    <joint name="base2trunk" type="fixed">
         <origin rpy="0 0 0" xyz="0 0 0"/>
         <parent link="base"/>

Commit message: adding intermediate ball link before wheel + using cylindrical collision for wheel to avoid discretization

File: robots/b2w_description/xacro/leg.xacro (robot description, xacro)
@@ -241,19 +241,46 @@
         </link>
         <xacro:if value="${ADD_WHEELS}">
+            <joint name="${name}_ball_joint" type="fixed">
+                <parent link="${name}_calf"/>
+                <child link="${name}_foot_ball"/>
+                <origin rpy="${-PI/2.0} 0.0 0.0" xyz="0.0 -0.001 -0.35"/>
+            </joint>
+            <link name="${name}_foot_ball">
+                <inertial>
+                    <origin xyz="0 0 0" rpy="0 0 0" />
+                    <mass value="0.1" />
+                    <inertia ixx="1E-04" ixy="0.0" ixz="0.0" iyy="1E-04" iyz="0.0" izz="1E-04" />
+                </inertial>
+                <visual>
+                    <origin rpy="0.0 0.0 0.0" xyz="0.0 0.0 0.0"/>
+                    <geometry>
+                        <sphere radius="0.05"/>
+                    </geometry>
+                    <material name="">
+                        <color rgba="1 1 1 1" />
+                    </material>
+                </visual>
+                <collision>
+                    <origin rpy="0.0 0.0 0.0" xyz="0.0 0.0 0.0"/>
+                    <geometry>
+                        <sphere radius="0.05"/>
+                    </geometry>
+                </collision>
+            </link>
             <joint name="${name}_foot_joint" type="continuous">
-                <origin xyz="0 -0.001 -0.35" rpy="0 0 0" />
-                <parent link="${name}_calf" />
+                <origin xyz="0 0 0" rpy="0 0 0" />
+                <parent link="${name}_foot_ball" />
                 <child link="${name}_foot" />
-                <axis xyz="0 1 0" />
+                <axis xyz="0 0 1" />
                 <limit effort="20" velocity="50" />
             </joint>
             <link name="${name}_foot">
                 <inertial>
-                    <origin xyz="-0.000991 -0.051053 -0.00113" rpy="0 0 0" />
+                    <origin xyz="-0.000991 -0.051053 -0.00113" rpy="${PI/2.0} 0 0" />
                     <mass value="1.083" />
                     <inertia ixx="0.004121" ixy="-6E-06" ixz="-4.8E-05" iyy="0.007776" iyz="-7E-06" izz="0.004108" />
                 </inertial>
                 <visual>
-                    <origin xyz="0 0 0" rpy="0 0 0" />
+                    <origin xyz="0 0 0" rpy="${PI/2.0} 0 0" />
                     <geometry>
                         <mesh filename="${MESH_PATH}/${name}_foot.dae" />
@@ -266,6 +293,10 @@
                     <origin xyz="0 0 0" rpy="0 0 0" />
                     <geometry>
+                        <cylinder radius="0.1125" length="0.03"/>
+                    </geometry>
+                    <!-- <origin xyz="0 0 0" rpy="${PI/2.0} 0 0" /> -->
+                    <!-- <geometry>
                         <mesh filename="${MESH_PATH}/${name}_foot.dae" />
-                    </geometry>
+                    </geometry> -->
                 </collision>
             </link>

Commit message: switched to stl filed for mujoco

File: robots/b2w_description/xacro/leg.xacro (robot description, xacro)
@@ -58,5 +58,5 @@
                 </xacro:if>
                 <geometry>
-                    <mesh filename="${MESH_PATH}/hip.dae" scale="1 1 1"/>
+                    <mesh filename="${MESH_PATH}/hip.stl" scale="1 1 1"/>
                 </geometry>
                 <material name="orange"/>
@@ -112,8 +112,8 @@
                 <geometry>
                     <xacro:if value="${mirror_dae == True}">
-                        <mesh filename="${MESH_PATH}/thigh.dae" scale="1 1 1"/>
+                        <mesh filename="${MESH_PATH}/thigh.stl" scale="1 1 1"/>
                     </xacro:if>
                     <xacro:if value="${mirror_dae == False}">
-                        <mesh filename="${MESH_PATH}/thigh_mirror.dae" scale="1 1 1"/>
+                        <mesh filename="${MESH_PATH}/thigh_mirror.stl" scale="1 1 1"/>
                     </xacro:if>
                 </geometry>
@@ -170,8 +170,8 @@
                 <geometry>
                     <xacro:if value="${mirror_dae == True}">
-                        <mesh filename="${MESH_PATH}/thigh.dae" scale="1 1 1"/>
+                        <mesh filename="${MESH_PATH}/thigh.stl" scale="1 1 1"/>
                     </xacro:if>
                     <xacro:if value="${mirror_dae == False}">
-                        <mesh filename="${MESH_PATH}/thigh_mirror.dae" scale="1 1 1"/>
+                        <mesh filename="${MESH_PATH}/thigh_mirror.stl" scale="1 1 1"/>
                     </xacro:if>
                 </geometry>
@@ -182,8 +182,8 @@
                 <geometry>
                     <xacro:if value="${mirror_dae == True}">
-                        <mesh filename="${MESH_PATH}/calf.dae" scale="1 1 1"/>
+                        <mesh filename="${MESH_PATH}/calf.stl" scale="1 1 1"/>
                     </xacro:if>
                     <xacro:if value="${mirror_dae == False}">
-                        <mesh filename="${MESH_PATH}/calf_mirror.dae" scale="1 1 1"/>
+                        <mesh filename="${MESH_PATH}/calf_mirror.stl" scale="1 1 1"/>
                     </xacro:if>
                 </geometry>
@@ -284,5 +284,5 @@
                     <origin xyz="0 0 0" rpy="${PI/2.0} 0 0" />
                     <geometry>
-                        <mesh filename="${MESH_PATH}/${name}_foot.dae" />
+                        <mesh filename="${MESH_PATH}/${name}_foot.stl" />
                     </geometry>
                     <material name="">
@@ -297,5 +297,5 @@
                     <!-- <origin xyz="0 0 0" rpy="${PI/2.0} 0 0" /> -->
                     <!-- <geometry>
-                        <mesh filename="${MESH_PATH}/${name}_foot.dae" />
+                        <mesh filename="${MESH_PATH}/${name}_foot.stl" />
                     </geometry> -->
                 </collision>

File: robots/b2w_description/xacro/robot.urdf.xacro (robot description, xacro)
@@ -66,7 +66,6 @@
             <origin rpy="0 0 0" xyz="0 0 0"/>
             <geometry>
-                <mesh filename="${MESH_PATH}/trunk.dae" scale="1 1 1"/>
+                <mesh filename="${MESH_PATH}/trunk.stl" scale="1 1 1"/>
             </geometry>
-            <!-- <material name="orange"/> -->
         </visual>
         <collision>
@@ -79,5 +78,5 @@
             <origin rpy="0 0 0" xyz="0 0 0"/>
             <geometry>
-                <mesh filename="package://b1_description/meshes/trunk.dae" scale="1 1 1"/>
+                <mesh filename="package://b1_description/meshes/trunk.stl" scale="1 1 1"/>
             </geometry>
         </collision> -->

Commit message: using visual for wheels collision
Signed-off-by: Andrea Patrizi <andreapatrizi1b6e6@gmail.com>

File: robots/b2w_description/xacro/leg.xacro (robot description, xacro)
@@ -269,5 +269,5 @@
             </link>
             <joint name="${name}_foot_joint" type="continuous">
-                <origin xyz="0 0 0" rpy="0 0 0" />
+                <origin xyz="0 0 0.0" rpy="0 0 0" />
                 <parent link="${name}_foot_ball" />
                 <child link="${name}_foot" />
@@ -291,8 +291,11 @@
                 </visual>
                 <collision>
-                    <origin xyz="0 0 0" rpy="0 0 0" />
-                    <geometry>
+                    <origin xyz="0 0 0" rpy="${PI/2.0} 0 0" />
+                    <geometry>
+                        <mesh filename="${MESH_PATH}/${name}_foot.stl" />
+                    </geometry>
+                    <!-- <geometry>
                         <cylinder radius="0.1125" length="0.03"/>
-                    </geometry>
+                    </geometry> -->
                     <!-- <origin xyz="0 0 0" rpy="${PI/2.0} 0 0" /> -->
                     <!-- <geometry>

Commit message: default to cylinders for wheel collisions
Signed-off-by: AndrePatri <andreapatrizi97@gmail.com>

File: robots/b2w_description/xacro/leg.xacro (robot description, xacro)
@@ -291,15 +291,12 @@
                 </visual>
                 <collision>
-                    <origin xyz="0 0 0" rpy="${PI/2.0} 0 0" />
-                    <geometry>
-                        <mesh filename="${MESH_PATH}/${name}_foot.stl" />
-                    </geometry>
-                    <!-- <geometry>
-                        <cylinder radius="0.1125" length="0.03"/>
-                    </geometry> -->
                     <!-- <origin xyz="0 0 0" rpy="${PI/2.0} 0 0" /> -->
                     <!-- <geometry>
                         <mesh filename="${MESH_PATH}/${name}_foot.stl" />
                     </geometry> -->
+                    <origin xyz="0 0 ${0.045*mirror}" rpy="0 0 0" />
+                    <geometry>
+                        <cylinder radius="0.1125" length="0.03"/>
+                    </geometry>
                 </collision>
             </link>
